Commit message: custom moveit config and urdfs for both gripper attachments

File: gen3_140_moveit_config/config/gen3.ros2_control.xacro (robot description, xacro)
@@ -10,4 +10,5 @@
             <joint name="joint_1">
                 <command_interface name="position"/>
+                <command_interface name="velocity"/>
                 <state_interface name="position">
                   <param name="initial_value">${initial_positions['joint_1']}</param>
@@ -17,4 +18,5 @@
             <joint name="joint_2">
                 <command_interface name="position"/>
+                <command_interface name="velocity"/>
                 <state_interface name="position">
                   <param name="initial_value">${initial_positions['joint_2']}</param>
@@ -24,4 +26,5 @@
             <joint name="joint_3">
                 <command_interface name="position"/>
+                <command_interface name="velocity"/>
                 <state_interface name="position">
                   <param name="initial_value">${initial_positions['joint_3']}</param>
@@ -31,4 +34,5 @@
             <joint name="joint_4">
                 <command_interface name="position"/>
+                <command_interface name="velocity"/>
                 <state_interface name="position">
                   <param name="initial_value">${initial_positions['joint_4']}</param>
@@ -38,4 +42,5 @@
             <joint name="joint_5">
                 <command_interface name="position"/>
+                <command_interface name="velocity"/>
                 <state_interface name="position">
                   <param name="initial_value">${initial_positions['joint_5']}</param>
@@ -45,4 +50,5 @@
             <joint name="joint_6">
                 <command_interface name="position"/>
+                <command_interface name="velocity"/>
                 <state_interface name="position">
                   <param name="initial_value">${initial_positions['joint_6']}</param>
@@ -52,4 +58,5 @@
             <joint name="finger_joint">
                 <command_interface name="position"/>
+                <command_interface name="velocity"/>
                 <state_interface name="position">
                   <param name="initial_value">${initial_positions['finger_joint']}</param>

File: gen3_85_moveit_config/config/gen3.urdf.xacro (robot description, xacro)
@@ -3,5 +3,5 @@
     <xacro:arg name="initial_positions_file" default="initial_positions.yaml" />
     <!-- Import gen3 urdf file -->
-    <xacro:include filename="$(find kortex_description)/robots/gen3.urdf" />
+    <xacro:include filename="$(find kortex_description)/robots/gen3_2f85.urdf" />
     <!-- Import control_xacro -->
     <xacro:include filename="gen3.ros2_control.xacro" />

File: kortex_description/arms/gen3/6dof/urdf/gen3_macro.xacro (robot description, xacro)
@@ -58,7 +58,7 @@
       <xacro:insert_block name="origin" />
       <parent link="${parent}"/>
-      <child link="${prefix}base_link" />
-    </joint>
-    <link name="${prefix}base_link">
+      <child link="${prefix}gen3_base_link" />
+    </joint>
+    <link name="${prefix}gen3_base_link">
       <inertial>
         <origin xyz="-0.000648 -0.000166 0.084487" rpy="0 0 0" />
@@ -69,14 +69,14 @@
         <origin xyz="0 0 0" rpy="0 0 0" />
         <geometry>
-          <mesh filename="file://$(find kortex_description)/arms/gen3/${dof}dof/meshes/base_link.STL" />
-        </geometry>
-        <material name="">
-          <color rgba="0.75294 0.75294 0.75294 1" />
-        </material>
-      </visual>
-      <collision>
-        <origin xyz="0 0 0" rpy="0 0 0" />
-        <geometry>
-          <mesh filename="file://$(find kortex_description)/arms/gen3/${dof}dof/meshes/base_link.STL" />
+          <mesh filename="package://kortex_description/arms/gen3/${dof}dof/meshes/base_link.STL" />
+        </geometry>
+        <material name="">
+          <color rgba="0.75294 0.75294 0.75294 1" />
+        </material>
+      </visual>
+      <collision>
+        <origin xyz="0 0 0" rpy="0 0 0" />
+        <geometry>
+          <mesh filename="package://kortex_description/arms/gen3/${dof}dof/meshes/base_link.STL" />
         </geometry>
       </collision>
@@ -91,14 +91,14 @@
         <origin xyz="0 0 0" rpy="0 0 0" />
         <geometry>
-          <mesh filename="file://$(find kortex_description)/arms/gen3/${dof}dof/meshes/shoulder_link.STL" />
-        </geometry>
-        <material name="">
-          <color rgba="0.75294 0.75294 0.75294 1" />
-        </material>
-      </visual>
-      <collision>
-        <origin xyz="0 0 0" rpy="0 0 0" />
-        <geometry>
-          <mesh filename="file://$(find kortex_description)/arms/gen3/${dof}dof/meshes/shoulder_link.STL" />
+          <mesh filename="package://kortex_description/arms/gen3/${dof}dof/meshes/shoulder_link.STL" />
+        </geometry>
+        <material name="">
+          <color rgba="0.75294 0.75294 0.75294 1" />
+        </material>
+      </visual>
+      <collision>
+        <origin xyz="0 0 0" rpy="0 0 0" />
+        <geometry>
+          <mesh filename="package://kortex_description/arms/gen3/${dof}dof/meshes/shoulder_link.STL" />
         </geometry>
       </collision>
@@ -111,5 +111,5 @@
           xyz="0 0 0.15643"
           rpy="-3.1416 0.0 0.0" />
-        <parent link="${prefix}base_link" />
+        <parent link="${prefix}gen3_base_link" />
         <child link="${prefix}shoulder_link" />
         <axis xyz="0 0 1" />
@@ -128,5 +128,5 @@
           xyz="0 0 0.15643"
           rpy="-3.1416 0.0 0.0" />
-        <parent link="${prefix}base_link" />
+        <parent link="${prefix}gen3_base_link" />
         <child link="${prefix}shoulder_link" />
         <axis xyz="0 0 1" />
@@ -155,5 +155,5 @@
           rpy="0 0 0" />
         <geometry>
-          <mesh filename="file://$(find kortex_description)/arms/gen3/${dof}dof/meshes/bicep_link.STL" />
+          <mesh filename="package://kortex_description/arms/gen3/${dof}dof/meshes/bicep_link.STL" />
         </geometry>
         <material name="">
@@ -166,5 +166,5 @@
           rpy="0 0 0" />
         <geometry>
-          <mesh filename="file://$(find kortex_description)/arms/gen3/${dof}dof/meshes/bicep_link.STL" />
+          <mesh filename="package://kortex_description/arms/gen3/${dof}dof/meshes/bicep_link.STL" />
         </geometry>
       </collision>
@@ -186,14 +186,14 @@
         <origin xyz="0 0 0" rpy="0 0 0" />
         <geometry>
-          <mesh filename="file://$(find kortex_description)/arms/gen3/${dof}dof/meshes/forearm_link.STL" />
-        </geometry>
-        <material name="">
-          <color rgba="0.75294 0.75294 0.75294 1" />
-        </material>
-      </visual>
-      <collision>
-        <origin xyz="0 0 0" rpy="0 0 0" />
-        <geometry>
-          <mesh filename="file://$(find kortex_description)/arms/gen3/${dof}dof/meshes/forearm_link.STL" />
+          <mesh filename="package://kortex_description/arms/gen3/${dof}dof/meshes/forearm_link.STL" />
+        </geometry>
+        <material name="">
+          <color rgba="0.75294 0.75294 0.75294 1" />
+        </material>
+      </visual>
+      <collision>
+        <origin xyz="0 0 0" rpy="0 0 0" />
+        <geometry>
+          <mesh filename="package://kortex_description/arms/gen3/${dof}dof/meshes/forearm_link.STL" />
         </geometry>
       </collision>
@@ -215,14 +215,14 @@
         <origin xyz="0 0 0" rpy="0 0 0" />
         <geometry>
-          <mesh filename="file://$(find kortex_description)/arms/gen3/${dof}dof/meshes/spherical_wrist_1_link.STL" />
-        </geometry>
-        <material name="">
-          <color rgba="0.75294 0.75294 0.75294 1" />
-        </material>
-      </visual>
-      <collision>
-        <origin xyz="0 0 0" rpy="0 0 0" />
-        <geometry>
-          <mesh filename="file://$(find kortex_description)/arms/gen3/${dof}dof/meshes/spherical_wrist_1_link.STL" />
+          <mesh filename="package://kortex_description/arms/gen3/${dof}dof/meshes/spherical_wrist_1_link.STL" />
+        </geometry>
+        <material name="">
+          <color rgba="0.75294 0.75294 0.75294 1" />
+        </material>
+      </visual>
+      <collision>
+        <origin xyz="0 0 0" rpy="0 0 0" />
+        <geometry>
+          <mesh filename="package://kortex_description/arms/gen3/${dof}dof/meshes/spherical_wrist_1_link.STL" />
         </geometry>
       </collision>
@@ -255,14 +255,14 @@
         <origin xyz="0 0 0" rpy="0 0 0" />
         <geometry>
-          <mesh filename="file://$(find kortex_description)/arms/gen3/${dof}dof/meshes/spherical_wrist_2_link.STL" />
-        </geometry>
-        <material name="">
-          <color rgba="0.75294 0.75294 0.75294 1" />
-        </material>
-      </visual>
-      <collision>
-        <origin xyz="0 0 0" rpy="0 0 0" />
-        <geometry>
-          <mesh filename="file://$(find kortex_description)/arms/gen3/${dof}dof/meshes/spherical_wrist_2_link.STL" />
+          <mesh filename="package://kortex_description/arms/gen3/${dof}dof/meshes/spherical_wrist_2_link.STL" />
+        </geometry>
+        <material name="">
+          <color rgba="0.75294 0.75294 0.75294 1" />
+        </material>
+      </visual>
+      <collision>
+        <origin xyz="0 0 0" rpy="0 0 0" />
+        <geometry>
+          <mesh filename="package://kortex_description/arms/gen3/${dof}dof/meshes/spherical_wrist_2_link.STL" />
         </geometry>
       </collision>
@@ -285,14 +285,14 @@
         <origin xyz="0 0 0" rpy="0 0 0" />
         <geometry>
-          <mesh filename="file://$(find kortex_description)/arms/gen3/${dof}dof/meshes/bracelet_with_vision_link.STL" />
-        </geometry>
-        <material name="">
-          <color rgba="0.75294 0.75294 0.75294 1" />
-        </material>
-      </visual>
-      <collision>
-        <origin xyz="0 0 0" rpy="0 0 0" />
-        <geometry>
-          <mesh filename="file://$(find kortex_description)/arms/gen3/${dof}dof/meshes/bracelet_with_vision_link.STL" />
+          <mesh filename="package://kortex_description/arms/gen3/${dof}dof/meshes/bracelet_with_vision_link.STL" />
+        </geometry>
+        <material name="">
+          <color rgba="0.75294 0.75294 0.75294 1" />
+        </material>
+      </visual>
+      <collision>
+        <origin xyz="0 0 0" rpy="0 0 0" />
+        <geometry>
+          <mesh filename="package://kortex_description/arms/gen3/${dof}dof/meshes/bracelet_with_vision_link.STL" />
         </geometry>
       </collision>
@@ -309,14 +309,14 @@
         <origin xyz="0 0 0" rpy="0 0 0" />
         <geometry>
-          <mesh filename="file://$(find kortex_description)/arms/gen3/${dof}dof/meshes/bracelet_no_vision_link.STL" />
-        </geometry>
-        <material name="">
-          <color rgba="0.75294 0.75294 0.75294 1" />
-        </material>
-      </visual>
-      <collision>
-        <origin xyz="0 0 0" rpy="0 0 0" />
-        <geometry>
-          <mesh filename="file://$(find kortex_description)/arms/gen3/${dof}dof/meshes/bracelet_no_vision_link.STL" />
+          <mesh filename="package://kortex_description/arms/gen3/${dof}dof/meshes/bracelet_no_vision_link.STL" />
+        </geometry>
+        <material name="">
+          <color rgba="0.75294 0.75294 0.75294 1" />
+        </material>
+      </visual>
+      <collision>
+        <origin xyz="0 0 0" rpy="0 0 0" />
+        <geometry>
+          <mesh filename="package://kortex_description/arms/gen3/${dof}dof/meshes/bracelet_no_vision_link.STL" />
         </geometry>
       </collision>

File: kortex_description/arms/gen3/7dof/urdf/gen3_macro.xacro (robot description, xacro)
@@ -59,7 +59,7 @@
       <xacro:insert_block name="origin" />
       <parent link="${parent}"/>
-      <child link="${prefix}base_link" />
+      <child link="${prefix}gen3_base_link" />
     </joint>
-    <link name="${prefix}base_link">
+    <link name="${prefix}gen3_base_link">
       <inertial>
         <origin xyz="-0.000648 -0.000166 0.084487" rpy="0 0 0" />

File: kortex_description/robots/gen3.xacro (robot description, xacro)
@@ -4,5 +4,5 @@
     <xacro:arg name="arm" default="gen3" />
     <xacro:arg name="dof" default="" />
-    <xacro:arg name="vision" default="false" />
+    <xacro:arg name="vision" default="true" />
     <xacro:arg name="robot_ip" default="192.168.11.11" />
     <xacro:arg name="username" default="admin" />
@@ -55,5 +55,47 @@
         use_external_cable="$(arg use_external_cable)"
         initial_positions="${xacro.load_yaml(initial_positions_file)}" >
-        <origin xyz="0 0 0" rpy="0 0 0" />  <!-- position robot in the world -->
+        <origin xyz="0.3 0 0.08" rpy="0 0 0" />  <!-- position robot in the world -->
     </xacro:load_robot>
+    <!--Back CB-->
+    <link name="rear_collision">
+    <visual>
+        <geometry>
+        <box size="0.55 0.10 0.10" />
+        </geometry>
+        <material name="red">
+        <color rgba="1 0 0 1" />
+        </material>
+    </visual>
+    <collision>
+        <geometry>
+        <box size="0.55 0.10 0.10" />
+        </geometry>
+    </collision>
+    </link>
+    <joint name="body_rear_collision" type="fixed">
+        <child link="rear_collision" />
+        <parent link="world" />
+        <origin xyz="-0.05 0 0.15" rpy="0 0 0" />
+    </joint>
+  <!-- Front CB -->
+  <link name="front_collision">
+    <visual>
+        <geometry>
+        <box size="0.10 0.10 0.10" />
+        </geometry>
+        <material name="red">
+        <color rgba="1 0 0 1" />
+        </material>
+    </visual>
+    <collision>
+        <geometry>
+        <box size="0.10 0.10 0.10" />
+        </geometry>
+    </collision>
+    </link>
+    <joint name="body_front_collision" type="fixed">
+        <child link="front_collision" />
+        <parent link="world" />
+        <origin xyz="0.42 0 0.125" rpy="0  0.3 0" />
+  </joint>
 </robot>

File: kortex_description/robots/gen3_2f140.urdf (robot description, URDF)
Before this commit: robot gen3, 24 links, 23 joints
Links:
- removed link left_finger_link
- removed link left_finger_tip_link
- removed link left_inner_knuckle_link
- removed link left_knuckle_link
- removed link right_finger_link
- removed link right_finger_tip_link
- removed link right_inner_knuckle_link
- removed link right_knuckle_link
- removed link robotiq_85_base_link
- added link left_inner_finger, mass 0.0104003125914103; collision mesh filename=package://robotiq_description/meshes/collision/2f_140/robot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; visual mesh filename=package://robotiq_description/meshes/visual/2f_140/robotiq_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
- added link left_inner_finger_pad; collision box size=0.03 0.07 0.0075; visual box size=0.027 0.065 0.0075
- added link left_inner_knuckle, mass 0.0271177346495152; collision mesh filename=package://robotiq_description/meshes/collision/2f_140/robot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; visual mesh filename=package://robotiq_description/meshes/visual/2f_140/robotiq_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
- added link left_outer_finger, mass 0.022614240507152; collision mesh filename=package://robotiq_description/meshes/collision/2f_140/robot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; visual mesh filename=package://robotiq_description/meshes/visual/2f_140/robotiq_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
- added link left_outer_knuckle, mass 0.00853198276973456; collision mesh filename=package://robotiq_description/meshes/collision/2f_140/robot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; visual mesh filename=package://robotiq_description/meshes/visual/2f_140/robotiq_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
- added link right_inner_finger, mass 0.0104003125914103; collision mesh filename=package://robotiq_description/meshes/collision/2f_140/robot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; visual mesh filename=package://robotiq_description/meshes/visual/2f_140/robotiq_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
- added link right_inner_finger_pad; collision box size=0.03 0.07 0.0075; visual box size=0.027 0.065 0.0075
- added link right_inner_knuckle, mass 0.0271177346495152; collision mesh filename=package://robotiq_description/meshes/collision/2f_140/robot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; visual mesh filename=package://robotiq_description/meshes/visual/2f_140/robotiq_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
- added link right_outer_finger, mass 0.022614240507152; collision mesh filename=package://robotiq_description/meshes/collision/2f_140/robot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; visual mesh filename=package://robotiq_description/meshes/visual/2f_140/robotiq_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
- added link right_outer_knuckle, mass 0.00853198276973456; collision mesh filename=package://robotiq_description/meshes/collision/2f_140/robot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; visual mesh filename=package://robotiq_description/meshes/visual/2f_140/robotiq_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
- added link robotiq_140_base_link, mass 0.22652; collision mesh filename=package://robotiq_description/meshes/collision/2f_140/robot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; visual mesh filename=package://robotiq_description/meshes/visual/2f_140/robotiq_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
Joints:
- removed joint left_finger_joint
- removed joint left_finger_tip_joint
- removed joint right_finger_joint
- removed joint right_finger_tip_joint
- removed joint right_knuckle_joint
- removed joint robotiq_85_base_joint
- added joint left_inner_finger_joint: type revolute, parent left_outer_finger, child left_inner_finger, origin xyz=0 0.0817554015893473 -0.0282203446692936 rpy=-0.725 0 0, axis 1 0 0, limit lower=-0.8757 upper=0.8757 effort=1000 velocity=2.0, mimic joint=finger_joint multiplier=1 offset=0
- added joint left_inner_finger_pad_joint: type fixed, parent left_inner_finger, child left_inner_finger_pad, origin xyz=0 0.0457554015893473 -0.0272203446692936 rpy=0 0 0, axis 0 0 1
- added joint left_outer_finger_joint: type fixed, parent left_outer_knuckle, child left_outer_finger, origin xyz=0 0.01821998610742 0.0260018192872234 rpy=0 0 0, axis 1 0 0
- added joint right_inner_finger_joint: type revolute, parent right_outer_finger, child right_inner_finger, origin xyz=0 0.0817554015893473 -0.0282203446692936 rpy=-0.725 0 0, axis 1 0 0, limit lower=-0.8757 upper=0.8757 effort=1000 velocity=2.0, mimic joint=finger_joint multiplier=1 offset=0
- added joint right_inner_finger_pad_joint: type fixed, parent right_inner_finger, child right_inner_finger_pad, origin xyz=0 0.0457554015893473 -0.0272203446692936 rpy=0 0 0, axis 0 0 1
- added joint right_outer_finger_joint: type fixed, parent right_outer_knuckle, child right_outer_finger, origin xyz=0 0.01821998610742 0.0260018192872234 rpy=0 0 0, axis 1 0 0
- added joint right_outer_knuckle_joint: type revolute, parent robotiq_140_base_link, child right_outer_knuckle, origin xyz=0 0.030601 0.054905 rpy=2.2957963267948966 0 3.141592653589793, axis 1 0 0, limit lower=-0.725 upper=0.725 effort=1000 velocity=2.0, mimic joint=finger_joint multiplier=-1 offset=0
- added joint robotiq_140_base_joint: type fixed, parent robotiq_base_link, child robotiq_140_base_link, origin xyz=0 0 0 rpy=0 0 0
- joint finger_joint: axis 0 -1 0 -> -1 0 0; child left_knuckle_link -> left_outer_knuckle; limit lower=0.0 upper=0.8 effort=50 velocity=0.5 -> lower=0 upper=0.72 effort=1000 velocity=2.0; origin xyz=0.03060114 0.0 0.05490452 rpy=0 0 0 -> xyz=0 -0.030601 0.054905 rpy=2.2957963267948966 0 0; parent robotiq_85_base_link -> robotiq_140_base_link
- joint joint_3: limit lower=-2.58 upper=2.58 effort=39 velocity=1.3963 -> lower=-2.57 upper=2.57 effort=39 velocity=1.3963
- joint left_inner_knuckle_joint: axis 0 -1 0 -> 1 0 0; child left_inner_knuckle_link -> left_inner_knuckle; limit (none) -> lower=-0.8757 upper=0.8757 effort=1000 velocity=2.0; mimic joint=finger_joint -> joint=finger_joint multiplier=-1 offset=0; origin xyz=0.0127 0.0 0.06142 rpy=0 0 0 -> xyz=0 -0.0127 0.06142 rpy=2.2957963267948966 0 0.0; parent robotiq_85_base_link -> robotiq_140_base_link; type continuous -> revolute
- joint right_inner_knuckle_joint: axis 0 -1 0 -> 1 0 0; child right_inner_knuckle_link -> right_inner_knuckle; limit (none) -> lower=-0.8757 upper=0.8757 effort=1000 velocity=2.0; mimic joint=finger_joint multiplier=-1 -> joint=finger_joint multiplier=-1 offset=0; origin xyz=-0.0127 0.0 0.06142 rpy=0 0 0 -> xyz=0 0.0127 0.06142 rpy=2.2957963267948966 0 -3.141592653589793; parent robotiq_85_base_link -> robotiq_140_base_link; type continuous -> revolute
- joint robotiq_base_joint: origin xyz=0 0 0 rpy=0 0 0 -> xyz=0 0 0 rpy=0 0 1.5707963267948966

File: kortex_description/robots/gen3_robotiq_2f_140.xacro (robot description, xacro)
@@ -3,18 +3,25 @@
     <!-- Arguments -->
     <xacro:arg name="arm" default="gen3" />
-    <xacro:arg name="dof" default="7" />
+    <xacro:arg name="dof" default="6" />
     <xacro:arg name="vision" default="true" />
     <xacro:arg name="gripper" default="robotiq_2f_140" />
     <xacro:arg name="use_internal_bus_gripper_comm" default="false" />
     <xacro:arg name="gripper_com_port" default="/dev/ttyUSB0" />
-    <xacro:arg name="sim" default="false" />
     <xacro:arg name="prefix" default="" />
     <xacro:include filename="$(find kortex_description)/robots/kortex_robot.xacro" />
     <xacro:load_robot
+      parent="base_link"
       arm="$(arg arm)"
       gripper="$(arg gripper)"
+      gripper_joint_name="gripper_base_joint"
       dof="$(arg dof)"
       vision="$(arg vision)"
-      sim="$(arg sim)"
+      robot_ip="192.168.50.9"
+      username="admin"
+      password="admin"
+      port="10000"
+      port_realtime="10001"
+      session_inactivity_timeout_ms="30000"
+      connection_inactivity_timeout_ms="30000"
       prefix="$(arg prefix)"
       use_internal_bus_gripper_comm="$(arg use_internal_bus_gripper_comm)"

File: kortex_description/robots/kinova.urdf.xacro (robot description, xacro)
@@ -7,5 +7,5 @@
   <xacro:arg name="arm" default="NO_ARM_TYPE_DEFINED" />
   <xacro:arg name="dof" default="7" />
-  <xacro:arg name="vision" default="false" />
+  <xacro:arg name="vision" default="true" />
   <xacro:arg name="robot_ip" default="192.168.11.11" />
   <xacro:arg name="username" default="admin" />
@@ -15,5 +15,5 @@
   <xacro:arg name="session_inactivity_timeout_ms" default="60000" />
   <xacro:arg name="connection_inactivity_timeout_ms" default="2000" />
-  <xacro:arg name="gripper" default="" />
+  <xacro:arg name="gripper" default="robotiq_2f_140" />
   <xacro:arg name="gripper_joint_name" default="finger_joint" />
   <xacro:arg name="gripper_max_velocity" default="100.0" />
@@ -64,5 +64,5 @@
     initial_positions="${xacro.load_yaml(initial_positions_file)}"
     moveit_active="$(arg moveit_active)">
-    <origin xyz="0 0 0" rpy="0 0 0" />  <!-- position robot in the world -->
+    <origin xyz="0.3 0 0.08" rpy="0 0 0" />  <!-- position robot in the world -->
   </xacro:load_robot>
   <xacro:if value="$(arg sim_gazebo)">
