Commit message: add moveit config for robotiq  85

File: gen3_85_moveit_config/config/gen3.urdf.xacro (robot description, xacro)
@@ -3,5 +3,5 @@
     <xacro:arg name="initial_positions_file" default="initial_positions.yaml" />
     <!-- Import gen3 urdf file -->
-    <xacro:include filename="$(find kortex_description)/robots/gen3_2f85.urdf" />
+    <xacro:include filename="$(find spot_description)/urdf/spot.urdf.xacro" />
     <!-- Import control_xacro -->
     <xacro:include filename="gen3.ros2_control.xacro" />

File: kortex_description/robots/gen3_2f85.urdf (robot description, URDF)
Before this commit: robot gen3, 24 links, 23 joints
Links:
- removed link front_collision
- removed link rear_collision
- removed link world
Joints:
- removed joint base_joint
- removed joint body_front_collision
- removed joint body_rear_collision
